Commit message: adding moveit file

File: src/open_manipulator_desp/urdf/open_manipulator.transmission.xacro (robot description, xacro)
@@ -18,5 +18,5 @@
       <type>transmission_interface/SimpleTransmission</type>
       <joint name="${joint}">
-        <hardwareInterface>hardware_interface/EffortJointInterface</hardwareInterface>
+        <hardwareInterface>hardware_interface/PositionJointInterface</hardwareInterface>
       </joint>
       <actuator name="motor${n}">

File: src/open_manipulator_desp/urdf/open_manipulator.urdf.xacro (robot description, xacro)
@@ -213,10 +213,10 @@
   </link>
   <!-- end effector joint -->
-  <joint name="end_effector_joint" type="fixed">
+  <!--<joint name="end_effector_joint" type="fixed">
     <origin xyz="0.126 0.0 0.0" rpy="0 0 0"/>
     <parent link="link5"/>
     <child link="end_effector_link"/>
   </joint>
-  <!-- end effector link -->
+  end effector link
   <link name="end_effector_link">
     <visual>
@@ -234,7 +234,7 @@
                izz="1.0e-03" />
     </inertial>
-  </link>
+  </link>-->
   <!-- Realsense Camera Joint Position -->
-  <joint name="camera_joint" type="fixed">
+  <!--<joint name="camera_joint" type="fixed">
     <axis xyz="0 1 0" />
     <origin xyz="0.070 0.032 0.052" rpy="0 0 0"/>
@@ -242,4 +242,4 @@
     <child link="camera_link"/>
   </joint>
-  <link name="camera_link"/>
+  <link name="camera_link"/> -->
 </robot>
